File: versions/v7-raw-34/v7-raw-34.kicad_sch (KiCad schematic)
At the start: 129 parts, among them J1 USB_C_Receptacle_USB2.0, J10 AXT-310124, J11 THD2528-11SD-GF, J12 SM04B-SRSS-TB_LF__SN_, J2 EXTENSION_HEADER, J3 USB_HDR, J5 CONN_BAT, J6 FH34SRJ-6S-0.5SH_99_, J7 ESP_HDR, J8 ESP_XTR_HDR, Q1 AO3401A, Q3 MMBT3904, Q4 MMBT3904, U1 RT9080-33GJ5, U10 ED060XC5, U11 TP4056, U12 RY3730, U2 PCA9535PW, U3 TPS651851RSLR, U4 USBLC6-2P6, U5 XC6206PxxxMR, U6 RY3730, U8 ESP32-S3-WROOM-1, U9 CH340C

Commit message: Add kindle 34 pins versions (RAW)
Parts:
- removed C45: 10uF, Capacitor_SMD:C_0805_2012Metric, symbol Device:C
- removed C46: 1uF/25V, Capacitor_SMD:C_0805_2012Metric, symbol Device:C
- removed D12: MBR0540, Diode_SMD:D_SOD-123, symbol Diode:MBR0540
- removed J10: AXT-310124, footprint:AXT310124, symbol FL_Paperwhite_AXT:AXT-310124
- removed J2: EXTENSION_HEADER, Connector_PinHeader_2.54mm:PinHeader_1x13_P2.54mm_Vertical, symbol Connector:Conn_01x13_Socket
- removed J5: CONN_BAT, Connector_PinHeader_2.54mm:PinHeader_1x02_P2.54mm_Vertical, symbol Connector:Conn_01x02_Socket
- removed J7: ESP_HDR, Connector_PinHeader_2.54mm:PinHeader_1x12_P2.54mm_Vertical, symbol Connector:Conn_01x12_Socket
- removed J8: ESP_XTR_HDR, Connector_PinHeader_2.54mm:PinHeader_1x05_P2.54mm_Vertical, symbol Connector:Conn_01x05_Socket
- removed L4: 22 uH, footprint:SWPA5040S282MT, symbol Device:L
- removed R16, R33: 10k, Resistor_SMD:R_0603_1608Metric, symbol Device:R
- removed R17: 25Ω, Resistor_SMD:R_0603_1608Metric, symbol Device:R
- removed R24 (x2): 33k, Resistor_SMD:R_0603_1608Metric, symbol Device:R
- removed R5: 0, Resistor_SMD:R_0603_1608Metric, symbol Device:R
- removed U12: RY3730, footprint:SOT-23-6_RY3730_Led_PWM, symbol FL_Led_driver:RY3730
- removed U2: PCA9535PW, Package_SO:TSSOP-24_4.4x7.8mm_P0.65mm, symbol Interface_Expansion:PCA9555PW
- added C21: C_Polarized 100uF, Capacitor_Tantalum_SMD:CP_EIA-3528-21_Kemet-B, symbol Device:C_Polarized
- added C39: 12 pF, Capacitor_SMD:C_0603_1608Metric, symbol Device:C
- added D12: 1N4148WS, Diode_SMD:D_SOD-323, symbol Diode:1N4148WS
- added J2: S2B-PH-SM4-TB_LF__SN_, footprint:S2BPHSM4TBLFSN, symbol BATTERY:S2B-PH-SM4-TB_LF__SN_
- added K1: HC-1.25-6PWT, footprint:CONN-SMD_6P-P1.25_HC-1.25-6PWT, symbol Soldered symbols:HC-1.25-6PWT
- added R12: 10k, Resistor_SMD:R_0603_1608Metric, symbol Device:R
- added R16, R5: 0R, Resistor_SMD:R_0603_1608Metric, symbol Soldered symbols:0603R
- added R17: 10 K, Resistor_SMD:R_0603_1608Metric, symbol Device:R_Small
- added U2: PCF8563T, Package_SO:SOIC-8_3.9x4.9mm_P1.27mm, symbol Timer_RTC:PCF8563T
- added Y1: Crystal_Small, footprint:Q13FC1350000400-Crystal, symbol Device:Crystal_Small
- C40: value 100nF -> 12 pF; footprint Capacitor_SMD:C_0805_2012Metric -> Capacitor_SMD:C_0603_1608Metric; LCSC C49678 -> C38523
- J6: footprint footprint:FH34SRJ6S05SH99_Mirrored -> footprint:C224194_6x1_FH34SRJ-6S-0.5SH50_HIR
- R3: value 3.8k -> 2.4k; LCSC C103591 -> C22940
- R8: value 1k -> 2.4k; LCSC C21190 -> C22940
- RN1: footprint footprint:RESN_F392JTCE_UNR_SD-pullup -> footprint:C425297_RES-ARRAY-SMD_0402-8P-L2.0-W1.0-BL
- TP7: value C2 -> RTC_INT; footprint TestPoint:TestPoint_Pad_D2.5mm -> TestPoint:TestPoint_Pad_D1.5mm
- U6: LCSC (none) -> C370887; LCSC Part C370887 -> (none)
Connections:
- net LEDC2_PWM is gone; now on net TPS_VCOM_CTRL: U8.20 (GPIO12/TOUCH12/ADC2_CH1/FSPICLK/FSPIIO6/SUBSPICLK)
- net TP_RST is gone; now on net EP_OE: U8.17 (GPIO9/TOUCH9/ADC1_CH8/FSPIHD/SUBSPIHD)
- net 3.3V: now also J12.2, RN1.1 (R1.1), RN1.2 (R2.1), RN1.3 (R3.1), RN1.4 (R4.1), D12.2 (A), K1.1, K1.2, R12.1, R17.1; no longer C40.1, J12.3, RN1.5 (R4.2), RN1.6 (R3.2), RN1.7 (R2.2), RN1.8 (R1.2)
- net EP_MODE: now also U8.18 (GPIO10/TOUCH10/ADC1_CH9/FSPICS0/FSPIIO4/SUBSPICS0)
- net GND: now also C40.1, J12.1, C21.2, C39.1, J2.2, K1.5, K1.6, K1.7 (SH), U2.4 (VSS); no longer C40.2, J12.4
- net GPIO_1: no longer J11.8 (DAT1)
- net GPIO_14: now also RN1.5 (R4.2); no longer RN1.3 (R3.1), U8.22 (GPIO14/TOUCH14/ADC2_CH3/FSPIWP/FSPIDQS/SUBSPIWP)
- net IO0: now also RN1.7 (R2.2); no longer RN1.1 (R1.1)
- net LEDC1_A: no longer J6.2
- net LEDC1_KA: no longer J6.5
- net LEDC1_PWM: now also U8.23 (GPIO21); no longer U8.19 (GPIO11/TOUCH11/ADC2_CH0/FSPID/FSPIIO5/SUBSPID)
- net SCL: now also J12.4, U2.6 (SCL); no longer J12.1
- net SDA: now also J12.3, U2.5 (SDA); no longer J12.2
- net TPS_PWRUP: now also U8.19 (GPIO11/TOUCH11/ADC2_CH0/FSPID/FSPIIO5/SUBSPID)
- net TPS_PWR_GOOD: now also U8.24 (GPIO47/SPICLK_P/SUBSPICLK_P_DIFF), R12.2; no longer R14.2
- net TPS_WAKEUP: now also U8.22 (GPIO14/TOUCH14/ADC2_CH3/FSPIWP/FSPIDQS/SUBSPIWP)
- net TPS_nINT: now also R14.2, U8.21 (GPIO13/TOUCH13/ADC2_CH2/FSPIQ/FSPIIO7/SUBSPIQ)
- net SD_CD: now reaches J11.9 (CD)
- net SD_CD: now also RN1.8 (R1.2)
- net BAT+ renamed VBAT
- net VBAT: now also J2.1
- removed net GPIO_10: J11.5 (CLX), RN1.2 (R2.1), U8.18 (GPIO10/TOUCH10/ADC1_CH9/FSPICS0/FSPIIO4/SUBSPICS0)
- removed net GPIO_13: J11.2 (CD/DAT3), RN1.4 (R4.1), U8.21 (GPIO13/TOUCH13/ADC2_CH2/FSPIQ/FSPIIO7/SUBSPIQ)
- net GPIO_2: no longer names the net of J11.1 (DAT2)
- net GPIO_2: no longer U8.38 (GPIO2/TOUCH2/ADC1_CH1)
- net GPIO_46 renamed RXD
- net RXD: now also R16.2
- net LEDC2_A: no longer names the net of J6.3
- net LEDC2_A: no longer TP7.1
- net LEDC2_KA: no longer names the net of J6.4
- net ~{GPIO_INTR} renamed GPIO_38
- net GPIO_38: now also J11.5 (CLX), RN1.6 (R3.2)
- new net: K1.4, R16.1
- new net: C39.2, U2.1 (OSCI), Y1.2
- new net: C21.1, D12.1 (K), U2.8 (VDD)
- new net: R17.2, TP7.1, U2.3 (~{INT})
- new net: C40.2, U2.2 (OSCO), Y1.1
- new net: K1.3, R5.1
- new net TXD: R5.2, U8.38 (GPIO2/TOUCH2/ADC1_CH1)
- no-connect marks 34 -> 31
Other:
- note added: "Battery Jack"
- note added: "Do we really need RTC_INT pin ?"
- note added: "FRONT LIGHT EC060XCD 6 pin"
- note added: "PCF8563T Real time clock via I2C"
- note added: "PSRAM < DO < NOT < USE"
- note added: "QWIIC Connector (TX / RX)"
- note added: "USB + / USB -"
- note removed: "ESP Header"
- note removed: "FRONT LIGHT EC060KH5 6 pin"
- note removed: "FRONT LIGHT ED060X** Paperwhite 10 pin AXE"
- note removed: "GPIO Expander with EPD + Power Controls"
- note removed: "Matching GROVE pinout"
- note removed: "QWIIC Connector (I2C)"
- note removed: "Warm"
- note removed: "{"
- moved on the sheet: J11, J12, J3, J6, RN1
