File: versions/v7-raw-34/v7-raw-34.kicad_sch (KiCad schematic)
At the start: 123 parts, among them J1 USB_C_Receptacle_USB2.0, J11 THD2528-11SD-GF, J12 SM04B-SRSS-TB_LF__SN_, J2 S2B-PH-SM4-TB_LF__SN_, J3 USB_HDR, J6 FH34SRJ-6S-0.5SH_99_, K1 HC-1.25-6PWT, Q1 AO3401A, Q3 MMBT3904, Q4 MMBT3904, U1 RT9080-33GJ5, U10 ED060XC5, U11 TP4056, U2 PCF8563T, U3 TPS651851RSLR, U4 USBLC6-2P6, U5 XC6206PxxxMR, U6 RY3730, U8 ESP32-S3-WROOM-1, U9 CH340C, Y1 Crystal_Small

Commit message: v7-raw 34
Parts:
- removed J3: USB_HDR, Connector_PinHeader_2.54mm:PinHeader_1x02_P2.54mm_Vertical, symbol Connector:Conn_01x02_Socket
- removed K1: HC-1.25-6PWT, footprint:CONN-SMD_6P-P1.25_HC-1.25-6PWT, symbol Soldered symbols:HC-1.25-6PWT
- removed R16, R5: 0R, Resistor_SMD:R_0603_1608Metric, symbol Soldered symbols:0603R
- added J3: Conn_01x04_Pin, Connector_PinHeader_2.54mm:PinHeader_1x04_P2.54mm_Vertical, symbol Connector:Conn_01x04_Pin
- added J4: USB_C_Receptacle_USB2.0, Connector_USB:USB_C_Receptacle_HRO_TYPE-C-31-M-12, symbol Connector:USB_C_Receptacle_USB2.0
Connections:
- net 3.3V: now also J3.4 (Pin_4)
- net ESP_USB+: now also J4.A6 (D+), J4.B6 (D+)
- net ESP_USB-: now also J4.A7 (D-), J4.B7 (D-)
- net GND: now also J3.1 (Pin_1), J4.A1 (GND), J4.A12 (GND), J4.B1 (GND), J4.B12 (GND), J4.S1 (SHIELD)
- net VBUS: now also J4.A4 (VBUS), J4.A9 (VBUS), J4.B4 (VBUS), J4.B9 (VBUS)
- net CC1: now reaches J1.A5 (CC1), R7.1
- net CC1: now also J4.A5 (CC1)
- net CC2: now reaches J1.B5 (CC2), R2.1
- net CC2: now also J4.B5 (CC2)
- net RXD renamed GPIO_46
- net GPIO_46: now also J3.2 (Pin_2)
- net TXD renamed GPIO_2
- net GPIO_2: now also J3.3 (Pin_3)
- no-connect marks 31 -> 33
Other:
- note added: "ADDITIONAL IOs"
- note added: "CDC USB"
- note added: "PROG USB"
- note removed: "USB + / USB -"
- note removed: "USB Connector"
- moved on the sheet: C16, C2, C3, D7, J2, Q1, R31, U1
