File: versions/v7-raw-34/v7-raw-34.kicad_pcb (KiCad board)
At the start: 4 copper layers, 138.9 x 104.6 mm, 123 parts, among them J1 USB_C_Receptacle_USB2.0, J11 THD2528-11SD-GF, J12 SM04B-SRSS-TB_LF__SN_, J2 S2B-PH-SM4-TB_LF__SN_, J3 USB_HDR, J6 FH34SRJ-6S-0.5SH_99_, K1 HC-1.25-6PWT, Q1 AO3401A, Q3 MMBT3904, Q4 MMBT3904, U1 RT9080-33GJ5, U10 ED060XC5, U11 TP4056, U2 PCF8563T, U3 TPS651851RSLR, U4 USBLC6-2P6, U5 XC6206PxxxMR, U6 RY3730, U8 ESP32-S3-WROOM-1, U9 CH340C, Y1 Crystal_Small

Commit message: v7-raw 34
Parts:
- removed K1: HC-1.25-6PWT, footprint:CONN-SMD_6P-P1.25_HC-1.25-6PWT
- removed R16, R5: 0R, Resistor_SMD:R_0603_1608Metric
- added J4: USB_C_Receptacle_USB2.0, Connector_USB:USB_C_Receptacle_HRO_TYPE-C-31-M-12, F.Cu at (63.0, 102.5)
- J3: value USB_HDR -> Conn_01x04_Pin; footprint Connector_PinHeader_2.54mm:PinHeader_1x02_P2.54mm_Vertical -> Connector_PinHeader_2.54mm:PinHeader_1x04_P2.54mm_Vertical
- moved J3 134.1 mm to (196.0, 95.1), turned to 0 degrees
- moved C36 12.4 mm to (173.7, 128.9), turned to 180 degrees
- moved R28 12.3 mm to (173.9, 131.0), turned to 180 degrees
- moved J6 11.7 mm to (172.4, 117.2), turned to 80 degrees
- moved R26 4.35 mm to (195.1, 133.2), turned to -90 degrees
- moved J11 2.99 mm to (66.6, 85.9)
- moved J1 1.24 mm to (63.0, 113.6)
Connections:
- net Net-(J1-CC1) renamed /CC1
- net Net-(J1-CC2) renamed /CC2
- J3 pad 1: /ESP_USB- -> GND
- J3 pad 2: /ESP_USB+ -> /GPIO_46
- U8 pad 16: RXD -> /GPIO_46
- U8 pad 38: TXD -> /GPIO_2
Routing:
- net /GPIO_2: track 0.00 -> 113.4 mm
- net TXD: track 107.2 -> 0.00 mm, vias 2 -> 0
- net /GPIO_46: track 0.00 -> 69.3 mm, vias 0 -> 2
- net RXD: track 57.4 -> 0.00 mm, vias 2 -> 0
- net VBUS: track 41.4 -> 62.5 mm, vias 3 -> 5
- net /CC1: track 6.38 -> 24.5 mm, vias 0 -> 2
- net /CC2: track 6.88 -> 23.0 mm
- net /LEDC1_KA: track 47.4 -> 36.6 mm
- net Net-(K1-Pad4): track 7.28 -> 0.00 mm
- net Net-(K1-Pad3): track 7.21 -> 0.00 mm
- net /LEDC1_A: track 61.4 -> 54.4 mm
- net 3.3V: track 195.6 -> 202.5 mm
- net /GPIO_38: track 77.3 -> 81.8 mm
- net /SD_CD: track 6.48 -> 10.8 mm
- net GND: track 180.8 -> 177.9 mm, vias 106 -> 104
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Other:
- board text added: "CDC"
- board text added: "PROG-UART"
- board text removed: "D+ IO20 D- IO19"
