File: epdiy-v7-light/epdiy-v7-light.kicad_pcb (KiCad board)
At the start: 4 copper layers, 110.8 x 68.5 mm, 117 parts, among them IC1 TPS2117DRLR, IC2 BQ27426YZFR, J2 EXTENSION_HEADER, J3 SM04B-SRSS-TB_LF__SN_, J4 Conn_01x02_Shielded, J9 USB_C_Receptacle_USB2.0, Q2 CPH3350, Q3 NTR4170NT1G, Q4 CPH3350, SW1 HX-3X6X3.5-CA-0.6-2.5N, SW2 HX-3X6X3.5-CA-0.6-2.5N, SW3 HX-3X6X3.5-CA-0.6-2.5N, SW4 HX-3X6X3.5-CA-0.6-2.5N, SW5 HX-3X6X3.5-CA-0.6-2.5N, SW6 MK-12C02-G015, U1 MCP1700-3302E_SOT23, U10 RT9080-33GJ5, U11 TP4056, U2 PCA9535PW, U3 TPS651851RSLR, U4 DS3231MZ, U6 ED078KH6, U8 ESP32-S3-WROOM-1

Commit message: Update RTC
Parts:
- added R32: 0Ω, Resistor_SMD:R_0603_1608Metric, F.Cu at (155.7, 86.5)
- SW2: value HX-3X6X3.5-CA-0.6-2.5N -> HX TS24CB 160GF; footprint footprints:SW-SMD_HX-3X6X3.5-CA-0.6-2.5N -> footprints:C25168832_TS24CB-160GF
- SW6: footprint footprints:C2911519_switch-MK-12C02-G020 -> footprints:C963206_MK-12C02-G020
- U4: value DS3231MZ -> RV-3032-C7 32.768KHZ-2.5PPM-TA-QC; footprint Package_SO:SOIC-8_3.9x4.9mm_P1.27mm -> footprints:C5127802_RV3032
- moved C14 2.67 mm to (155.7, 84.0)
- moved U4 1.74 mm to (156.6, 74.1)
- moved SW6 0.20 mm to (169.9, 69.3)
- moved SW2 0.12 mm to (152.4, 89.6)
Connections:
- SW2 pad 1: /EN -> Net-(R32-Pad1)
- U4 pad 2: +BATT -> /SDA
- U4 pad 6: unconnected-(U4-VBAT-Pad6) -> +BATT
- U4 pad 7: /SDA -> unconnected-(U4-CLKOUT-Pad7)
Routing:
- net /BTN_SELECT: track 73.7 -> 68.2 mm
- net GND: track 178.7 -> 173.5 mm, vias 102 -> 105
- net /SCL: track 210.5 -> 205.6 mm
- net /SDA: track 209.6 -> 206.0 mm
- net VIN2: track 35.8 -> 39.0 mm
- net /EN: track 30.0 -> 27.0 mm
- net RTC_INT: track 35.7 -> 38.0 mm
- net Net-(R32-Pad1): track 0.00 -> 2.07 mm
- net +BATT: track 138.4 -> 136.5 mm
- net PWR_HOLD: track 45.8 -> 46.9 mm
Other:
- outline, holes or cut-outs redrawn
- board text added: "Rel 1.0 PCB custom modified for 10.3 inch displays (16 bit) ED103TC* ED103M**"
- board text removed: "Rel 1.1.1 PCB custom modified for 9.7, 13.3 inch displays (8 bit)"
