File: epdiy-v7-light/epdiy-v7-light.kicad_sch (KiCad schematic)
At the start: 116 parts, among them IC1 TPS2117DRLR, IC2 BQ27426YZFR, J2 EXTENSION_HEADER, J3 SM04B-SRSS-TB_LF__SN_, J4 Conn_01x02_Shielded, J9 USB_C_Receptacle_USB2.0, Q2 CPH3350, Q3 NTR4170NT1G, Q4 CPH3350, SW1 HX-3X6X3.5-CA-0.6-2.5N, SW2 HX-3X6X3.5-CA-0.6-2.5N, SW3 HX-3X6X3.5-CA-0.6-2.5N, SW4 HX-3X6X3.5-CA-0.6-2.5N, SW5 HX-3X6X3.5-CA-0.6-2.5N, SW6 MK-12C02-G015, U1 MCP1700-3302E_SOT23, U10 RT9080-33GJ5, U11 TP4056, U2 PCA9535PW, U3 TPS651851RSLR, U4 DS3231MZ, U6 ED078KH6, U8 ESP32-S3-WROOM-1

Commit message: Update RTC
Parts:
- removed SW2: HX-3X6X3.5-CA-0.6-2.5N, footprints:SW-SMD_HX-3X6X3.5-CA-0.6-2.5N, symbol easyeda:HX-3X6X3.5-CA-0.6-2.5N
- removed U4: DS3231MZ, Package_SO:SOIC-8_3.9x4.9mm_P1.27mm, symbol Timer_RTC:DS3231MZ
- added R32: 0Ω, Resistor_SMD:R_0603_1608Metric, symbol Device:R
- added SW2: HX TS24CB 160GF, footprints:C25168832_TS24CB-160GF, symbol easyeda:HXTS24CB160GF
- added U4: RV-3032-C7 32.768KHZ-2.5PPM-TA-QC, footprints:C5127802_RV3032, symbol EASYEDA:RV-3032-C732.768KHZ-2.5PPM-TA-QC
- SW6: footprint footprints:C2911519_switch-MK-12C02-G020 -> footprints:C963206_MK-12C02-G020; LCSC C2911519 -> C963206
- U8: now left out of the parts list
Connections:
- net +BATT: now also U4.6 (VDD)
- net EN: now also R32.2
- net GND: now also SW2.2, U4.5 (VSS)
- net RTC_INT: now also U4.3 (~{INT})
- net SCL: now also U4.8 (SCL)
- net SDA: now also U4.2 (SDA)
- new net: R32.1, SW2.1
- no-connect marks 26 -> 27
