File: epdiy-v7-raw/epdiy-v7-raw.kicad_pcb (KiCad board)
At the start: 4 copper layers, 128.4 x 74.9 mm, 118 parts, among them CN1 WP27D-S050VA3-R15000, IC1 MPU-6500, J1 USB_C_Receptacle_USB2.0, J2 EXTENSION_HEADER, J3 SIGNALS_HEADER, J5 CONN_BAT, J6 THD2528-11SD-GF, J7 ESP_HDR, Q1 AO3401A, SW1 TC-0522C-1.7-160G, SW2 TC-0522C-1.7-160G, SW3 K2-1806SQ-A2DW-04, SW4 K2-1806SQ-A2DW-04, SW5 K2-1806SQ-A2DW-04, U1 RT9080-33GJ5, U10 ED060XC5, U11 TP4056, U3 TPS651851RSLR, U4 USBLC6-2P6, U8 ESP32-S3-WROOM-1, Y1 RV-3032-C7

Commit message: v7 raw corrections
Parts:
- moved R14 2.59 mm to (62.6, 58.8)
- moved R12 1.84 mm to (179.1, 113.9)
- moved R15 1.14 mm to (62.6, 73.2)
Routing:
- net Net-(R15-Pad1): track 2.08 -> 0.00 mm
- net GND: track 213.9 -> 212.2 mm, vias 102 -> 101
- net Net-(R12-Pad1): track 2.15 -> 3.58 mm
Other:
- board text added: "PROUDLY BUILT WITH LARRY BANK: https://github.com/bitbank2/FastEPD TEAM: @martinberlin @bitbank2"
- board text added: "Rel 1.1"
- board text removed: "RESEARCH LAB CATALUNYA HQ https://github.com/bitbank2/FastEPD TEAM: @martinberlin @bitbank2"
- board text removed: "Rel 1.0"
